File: pcb/owl-driver-board.kicad_sch (KiCad schematic)
At the start: 168 parts, among them J1 CONN_04, J10 1890963, J11 ENABLE, J2 RASPBERRYPI-40-PIN-GPIO, J3 1890963, J4 1890963, J5 1890963, J6 CONN_04X2, J7 1890963, J8 1890963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

Commit message: 4-way board, revision v2.5
Bump the revision with some small tweaks -
 - Lower profile Phoenix Contact screw terminals - replace 1890963 with 1935161 (C3819953)
 - 10k discharge resistor across all outputs to reduce ghost voltages
 - Format updates for KiCad 9
Parts:
- added R59, R60, R61, R62: 10k, Resistor_SMD:R_0603_1608Metric, symbol Device:R_US
- C8: now not fitted; now left out of the parts list
- D17, D2, D3, D6: value BZT52C5V1T -> BZT585B13T-7 13V; LCSC C2987034 -> C460799; Part (none) -> BZT585B13T-7
- D18: value BZT52C5V1T -> BZT585B13T-7 13V; LCSC C2987034 -> C460799; Note 9V Zener -> (none); Part (none) -> BZT585B13T-7
- J10, J3, J4, J5, J7, J8: value 1890963 -> 1935161; footprint misc:Connector_Phoenix-Contact_MKDSN_1890963_P5.0_2x -> TerminalBlock_Phoenix:TerminalBlock_Phoenix_PT-1,5-2-5.0-H_1x02_P5.00mm_Horizontal; LCSC C3817236 -> C3819953; Part (none) -> 1935161
Connections:
- net GND: now also R59.1, R60.1, R61.1, R62.1
- net M1_D: now also R62.2
- net M2_D: now also R61.2
- net M3_D: now also R60.2
- net M4_D: now also R59.2
Other:
- note added: "Alternative MOSFET AGM60P30AP / C20625923 Over specced but a little more expensive"
- note added: "Was Phoenix Contact part #1890963 (15mm height) Now part #1935161 (11mm height)"
- moved on the sheet: D19, D20, D4, D5, F2, F3, F4, F5, R15, R16, R4, R5
